Commit message: 231018

File: legged_examples/legged_unitree/legged_unitree_description/urdf/aliengoZ1/const.xacro (robot description, xacro)
@@ -204,15 +204,15 @@
     <xacro:property name="jointFriction" value="1.0"/>
     <xacro:property name="torqueMax" value="30.0"/>
-    <xacro:property name="velocityMax" value="10"/>
+    <xacro:property name="velocityMax" value="${PI}"/>
     <xacro:property name="joint1_PositionMin" value="${-PI*150/180}"/>
     <xacro:property name="joint1_PositionMax" value="${PI*150/180}"/>
     <xacro:property name="joint2_PositionMin" value="0.0"/>
     <xacro:property name="joint2_PositionMax" value="${PI}"/>
-    <xacro:property name="joint3_PositionMin" value="${-PI*274/180}"/>
+    <xacro:property name="joint3_PositionMin" value="${-PI*165/180}"/>
     <xacro:property name="joint3_PositionMax" value="0.0"/>
-    <xacro:property name="joint4_PositionMin" value="${-PI*100/180}"/>
-    <xacro:property name="joint4_PositionMax" value="${PI*90/180}"/>
-    <xacro:property name="joint5_PositionMin" value="${-PI*99/180}"/>
-    <xacro:property name="joint5_PositionMax" value="${PI*99/180}"/>
+    <xacro:property name="joint4_PositionMin" value="${-PI*80/180}"/>
+    <xacro:property name="joint4_PositionMax" value="${PI*80/180}"/>
+    <xacro:property name="joint5_PositionMin" value="${-PI*85/180}"/>
+    <xacro:property name="joint5_PositionMax" value="${PI*85/180}"/>
     <xacro:property name="joint6_PositionMin" value="${-PI*160/180}"/>
     <xacro:property name="joint6_PositionMax" value="${PI*160/180}"/>

Commit message: 2311011017

File: legged_examples/legged_unitree/legged_unitree_description/urdf/aliengoZ1/const.xacro (robot description, xacro)
@@ -205,16 +205,16 @@
     <xacro:property name="torqueMax" value="30.0"/>
     <xacro:property name="velocityMax" value="${PI}"/>
-    <xacro:property name="joint1_PositionMin" value="${-PI*150/180}"/>
-    <xacro:property name="joint1_PositionMax" value="${PI*150/180}"/>
+    <xacro:property name="joint1_PositionMin" value="${-PI*140/180}"/>
+    <xacro:property name="joint1_PositionMax" value="${PI*140/180}"/>
     <xacro:property name="joint2_PositionMin" value="0.0"/>
-    <xacro:property name="joint2_PositionMax" value="${PI}"/>
-    <xacro:property name="joint3_PositionMin" value="${-PI*165/180}"/>
+    <xacro:property name="joint2_PositionMax" value="${PI*170/180}"/>
+    <xacro:property name="joint3_PositionMin" value="${-PI*155/180}"/>
     <xacro:property name="joint3_PositionMax" value="0.0"/>
-    <xacro:property name="joint4_PositionMin" value="${-PI*80/180}"/>
-    <xacro:property name="joint4_PositionMax" value="${PI*80/180}"/>
-    <xacro:property name="joint5_PositionMin" value="${-PI*85/180}"/>
-    <xacro:property name="joint5_PositionMax" value="${PI*85/180}"/>
-    <xacro:property name="joint6_PositionMin" value="${-PI*160/180}"/>
-    <xacro:property name="joint6_PositionMax" value="${PI*160/180}"/>
+    <xacro:property name="joint4_PositionMin" value="${-PI*70/180}"/>
+    <xacro:property name="joint4_PositionMax" value="${PI*70/180}"/>
+    <xacro:property name="joint5_PositionMin" value="${-PI*75/180}"/>
+    <xacro:property name="joint5_PositionMax" value="${PI*75/180}"/>
+    <xacro:property name="joint6_PositionMin" value="${-PI*150/180}"/>
+    <xacro:property name="joint6_PositionMax" value="${PI*150/180}"/>
     <xacro:property name="Gripper_PositionMin" value="${-PI*90/180}"/>
     <xacro:property name="Gripper_PositionMax" value="0.0"/>
